File: Rov/comms.kicad_sch (KiCad schematic)
At the start: 3 parts, among them U1 DHT11, U2 MAX485E, U3 MAX485E

Commit message: Added more wiring
Parts:
- removed U1: DHT11, Sensor:Aosong_DHT11_5.5x12.0_P2.54mm, symbol Sensor:DHT11
Connections:
- net TX: now reaches U2.1 (RO)
- net GND: now reaches U2.2 (~{RE})
- net GND: now also U2.3 (DE), U2.5 (GND), U3.5 (GND)
- net VCC: now reaches U2.8 (VCC)
- net VCC: now also U3.2 (~{RE}), U3.3 (DE), U3.8 (VCC)
- net RX: now reaches U3.4 (DI)
Changed lines of the file:
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@@
 (kicad_sch (version 20230121) (generator eeschema)
   (paper "A4")
-  (wire (pts (xy 121.92 133.35) (xy 116.84 133.35))
+  (junction (at 111.76 119.38) (diameter 0) (color 0 0 0 0)
+  )
+  (junction (at 97.79 97.79) (diameter 0) (color 0 0 0 0)
+  )
+  (junction (at 107.95 119.38) (diameter 0) (color 0 0 0 0)
+  )
+  (junction (at 97.79 82.55) (diameter 0) (color 0 0 0 0)
+  )
+  (junction (at 111.76 82.55) (diameter 0) (color 0 0 0 0)
+  )
+  (wire (pts (xy 121.92 67.31) (xy 121.92 68.58))
+    (stroke (width 0) (type default))
+  )
+  (wire (pts (xy 107.95 119.38) (xy 111.76 119.38))
+    (stroke (width 0) (type default))
+  )
+  (wire (pts (xy 93.98 82.55) (xy 97.79 82.55))
+    (stroke (width 0) (type default))
+  )
+  (wire (pts (xy 97.79 133.35) (xy 121.92 133.35))
     (stroke (width 0) (type default))
   )
@@
     (stroke (width 0) (type default))
   )
+  (wire (pts (xy 97.79 82.55) (xy 97.79 97.79))
+    (stroke (width 0) (type default))
+  )
+  (wire (pts (xy 97.79 133.35) (xy 97.79 97.79))
+    (stroke (width 0) (type default))
+  )
   (wire (pts (xy 132.08 86.36) (xy 135.89 86.36))
+    (stroke (width 0) (type default))
+  )
+  (wire (pts (xy 111.76 119.38) (xy 111.76 120.65))
+    (stroke (width 0) (type default))
+  )
+  (wire (pts (xy 97.79 82.55) (xy 111.76 82.55))
+    (stroke (width 0) (type default))
+  )
+  (wire (pts (xy 107.95 105.41) (xy 107.95 119.38))
+    (stroke (width 0) (type default))
+  )
+  (wire (pts (xy 106.68 123.19) (xy 111.76 123.19))
     (stroke (width 0) (type default))
   )
@@
     (stroke (width 0) (type default))
   )
-  (wire (pts (xy 116.84 97.79) (xy 121.92 97.79))
+  (wire (pts (xy 97.79 97.79) (xy 121.92 97.79))
+    (stroke (width 0) (type default))
+  )
+  (wire (pts (xy 111.76 82.55) (xy 111.76 83.82))
+    (stroke (width 0) (type default))
+  )
+  (wire (pts (xy 111.76 78.74) (xy 106.68 78.74))
+    (stroke (width 0) (type default))
+  )
+  (wire (pts (xy 111.76 118.11) (xy 111.76 119.38))
+    (stroke (width 0) (type default))
+  )
+  (wire (pts (xy 111.76 81.28) (xy 111.76 82.55))
+    (stroke (width 0) (type default))
+  )
+  (wire (pts (xy 106.68 119.38) (xy 107.95 119.38))
     (stroke (width 0) (type default))
   )
@@
     (stroke (width 0) (type default))
   )
+  (wire (pts (xy 111.76 67.31) (xy 121.92 67.31))
+    (stroke (width 0) (type default))
+  )
+  (wire (pts (xy 121.92 105.41) (xy 107.95 105.41))
+    (stroke (width 0) (type default))
+  )
+  (hierarchical_label "VCC" (shape input) (at 111.76 67.31 180) (fields_autoplaced)
+    (effects (font (size 1.27 1.27)) (justify right))
+  )
   (hierarchical_label "TX_B" (shape output) (at 135.89 115.57 0) (fields_autoplaced)
     (effects (font (size 1.27 1.27)) (justify left))
+  )
+  (hierarchical_label "VCC" (shape input) (at 106.68 119.38 180) (fields_autoplaced)
+    (effects (font (size 1.27 1.27)) (justify right))
+  )
+  (hierarchical_label "RX" (shape input) (at 106.68 123.19 180) (fields_autoplaced)
+    (effects (font (size 1.27 1.27)) (justify right))
   )
   (hierarchical_label "RX_B" (shape output) (at 135.89 78.74 0) (fields_autoplaced)
     (effects (font (size 1.27 1.27)) (justify left))
   )
+  (hierarchical_label "GND" (shape input) (at 93.98 82.55 180) (fields_autoplaced)
+    (effects (font (size 1.27 1.27)) (justify right))
+  )
   (hierarchical_label "TX_A" (shape output) (at 135.89 123.19 0) (fields_autoplaced)
     (effects (font (size 1.27 1.27)) (justify left))
+  )
+  (hierarchical_label "TX" (shape output) (at 106.68 78.74 180) (fields_autoplaced)
+    (effects (font (size 1.27 1.27)) (justify right))
   )
   (hierarchical_label "RX_A" (shape output) (at 135.89 86.36 0) (fields_autoplaced)
@@
         )
       )
-    )
-  )
-  (symbol (lib_id "Sensor:DHT11") (at 123.19 52.07 0) (unit 1)
-    (in_bom yes) (on_board yes) (dnp no) (fields_autoplaced)
-    (property "Reference" "U1" (at 116.84 51.435 0)
-      (effects (font (size 1.27 1.27)) (justify right))
-    )
-    (property "Value" "DHT11" (at 116.84 53.975 0)
-      (effects (font (size 1.27 1.27)) (justify right))
-    )
-    (property "Footprint" "Sensor:Aosong_DHT11_5.5x12.0_P2.54mm" (at 123.19 62.23 0)
-      (effects (font (size 1.27 1.27)) hide)
-    )
-    (property "Datasheet" "http://akizukidenshi.com/download/ds/aosong/DHT11.pdf" (at 127 45.72 0)
-      (effects (font (size 1.27 1.27)) hide)
-    )
-    (pin "1")
-    (pin "2")
-    (pin "3")
-    (pin "4")
-    (instances
-      (project "Rov"
-        (path "/195799e7-2545-43ed-8a08-3008b09b45b7"
-          (reference "U1") (unit 1)
-        )
-        (path "/195799e7-2545-43ed-8a08-3008b09b45b7/02be91a2-af96-420c-a76d-c2f8801e0b9e"
-          (reference "U3") (unit 1)
-        )
-      )
